File: Pot-timed/LED-strip_PWM.kicad_pcb (KiCad board)
At the start: 2 copper layers, 29.7 x 10 mm, 16 parts, among them IC1 ATTINY13A-MM, P1 CONN_2, P2 CONN_2, T1 AO3400, U1 MCP1804-SOT23-5

Commit message: Changed to custom attiny13 schematic symbol + footprint.
Parts:
- IC1: value ATTINY13A-MM -> MADW__ATTINY13-MM
Connections:
- IC1 pad 3: (no net) -> N-000005
- IC1 pad 8: (no net) -> N-000006
Changed lines of the file:
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@@
-(kicad_pcb (version 3) (host pcbnew "(2013-05-28 BZR 4174)-testing")
+(kicad_pcb (version 3) (host pcbnew "(2013-06-07 BZR 4197)-testing")
   (general
     (links 31)
     (no_connects 0)
-    (area 74.5076 46.6476 111.616669 61.100001)
+    (area 75.899999 47.899999 105.750001 58.100001)
     (thickness 1.6002)
     (drawings 14)
@@
     (zones 0)
     (modules 16)
-    (nets 13)
+    (nets 15)
   )
   (page User 431.8 279.4)
@@
   (net 10 GNDPWR)
   (net 11 N-000004)
-  (net 12 VCC)
+  (net 12 N-000005)
+  (net 13 N-000006)
+  (net 14 VCC)
   (net_class Default "This is the default net class."
     (clearance 0.1524)
@@
     (add_net /drain)
     (add_net N-000004)
+    (add_net N-000005)
+    (add_net N-000006)
   )
   (net_class Power ""
@@
       (effects (font (size 1 1) (thickness 0.2)))
     )
-    (fp_text value ATTINY13A-MM (at 0 3.3) (layer F.SilkS) hide
+    (fp_text value MADW__ATTINY13-MM (at 0 3.3) (layer F.SilkS) hide
       (effects (font (size 1 1) (thickness 0.2)))
     )
@@
     (pad 3 smd rect (at -1.5 0) (size 1 0.25)
       (layers Front F.Paste F.Mask)
+      (net 12 N-000005)
     )
     (pad 4 smd rect (at -1.5 0.5) (size 1 0.25)
@@
     (pad 8 smd rect (at 1.5 0) (size 1 0.25)
       (layers Front F.Paste F.Mask)
+      (net 13 N-000006)
     )
     (pad 9 smd rect (at 1.5 -0.5) (size 1 0.25)
@@
     (pad 10 smd rect (at 1.5 -1) (size 1 0.25)
       (layers Front F.Paste F.Mask)
-      (net 12 VCC)
+      (net 14 VCC)
     )
   )
@@
     (pad 1 smd rect (at -0.94996 0) (size 1.29794 1.4986)
       (layers Front F.Paste F.Mask)
-      (net 12 VCC)
+      (net 14 VCC)
     )
     (pad 2 smd rect (at 0.94996 0) (size 1.29794 1.4986)
@@
     (pad 1 smd rect (at -0.94996 0) (size 1.29794 1.4986)
       (layers Front F.Paste F.Mask)
-      (net 12 VCC)
+      (net 14 VCC)
     )
     (pad 2 smd rect (at 0.94996 0) (size 1.29794 1.4986)
@@
     (pad 1 smd rect (at -1.00076 1.80086 90) (size 1.19888 1.19888)
       (layers Front F.Paste F.Mask)
-      (net 12 VCC)
+      (net 14 VCC)
     )
     (pad 3 smd rect (at 1.00076 1.80086 90) (size 1.19888 1.19888)
@@
     (pad 3 smd rect (at 1.00076 1.80086 90) (size 1.19888 1.19888)
       (layers Front F.Paste F.Mask)
-      (net 12 VCC)
+      (net 14 VCC)
     )
     (pad 2 smd rect (at 0 -1.45034 90) (size 1.6002 1.50114)
@@
     (pad 5 smd rect (at -0.95 -1.3) (size 0.65 1.25)
       (layers Front F.Paste F.Mask)
-      (net 12 VCC)
+      (net 14 VCC)
     )
   )
@@
     (pad 2 thru_hole oval (at -1.27 -0.635 180) (size 1.05 1.5) (drill 0.65 (offset 0 -0.2))
       (layers *.Cu *.Mask F.SilkS)
-      (net 12 VCC)
+      (net 14 VCC)
     )
     (pad 3 thru_hole oval (at 0 0.635 180) (size 1.05 1.5) (drill 0.65 (offset 0 0.2))
@@
   (segment (start 82.99982 53.94996) (end 82.99982 56.34854) (width 0.1524) (layer Front) (net 11) (status 30))
   (segment (start 82.99982 56.34854) (end 82.74836 56.6) (width 0.2032) (layer Front) (net 11) (status 30))
-  (segment (start 89.00086 52.00076) (end 90.00076 52.00076) (width 0.1524) (layer Back) (net 12))
-  (segment (start 90.00076 52.00076) (end 90.745198 52.745198) (width 0.1524) (layer Back) (net 12))
-  (segment (start 90.745198 52.745198) (end 93.754802 52.745198) (width 0.1524) (layer Back) (net 12))
-  (segment (start 93.754802 52.745198) (end 94.22 52.28) (width 0.1524) (layer Back) (net 12))
-  (segment (start 94.22 52.28) (end 94.22 51.335) (width 0.1524) (layer Back) (net 12))
-  (via (at 89.00086 52.00076) (size 0.635) (layers Front Back) (net 12) (status 30))
-  (segment (start 89.00086 54.29924) (end 89.00086 52.00076) (width 0.1524) (layer Front) (net 12) (status 30))
-  (segment (start 94.22 51.335) (end 96.735 51.335) (width 0.1524) (layer Back) (net 12) (status 10))
-  (via (at 97.4 52) (size 0.635) (layers Front Back) (net 12) (status 30))
-  (segment (start 97.4 52) (end 97.4 51.99996) (width 0.1524) (layer Front) (net 12) (status 30))
-  (segment (start 97.4 51.99996) (end 97.35004 51.95) (width 0.1524) (layer Front) (net 12) (status 30))
-  (segment (start 96.735 51.335) (end 97.4 52) (width 0.1524) (layer Back) (net 12))
-  (segment (start 94.45 54.2) (end 96.7 54.2) (width 0.1524) (layer Front) (net 12) (status 30))
-  (segment (start 96.7 54.2) (end 96.85 54.05) (width 0.3048) (layer Front) (net 12) (status 30))
-  (segment (start 97.35004 51.95) (end 97.35004 52.59996) (width 0.1524) (layer Front) (net 12) (status 30))
-  (segment (start 96.85 53.1) (end 96.85 54.05) (width 0.1524) (layer Front) (net 12) (status 20))
-  (segment (start 97.35004 52.59996) (end 96.85 53.1) (width 0.1524) (layer Front) (net 12) (status 10))
-  (segment (start 97.35004 49.45) (end 97.35004 51.95) (width 0.1524) (layer Front) (net 12) (status 30))
-  (segment (start 97.2 51.79996) (end 97.35004 51.95) (width 0.3048) (layer Front) (net 12) (status 30))
+  (segment (start 89.00086 52.00076) (end 90.00076 52.00076) (width 0.1524) (layer Back) (net 14))
+  (segment (start 90.00076 52.00076) (end 90.745198 52.745198) (width 0.1524) (layer Back) (net 14))
+  (segment (start 90.745198 52.745198) (end 93.754802 52.745198) (width 0.1524) (layer Back) (net 14))
+  (segment (start 93.754802 52.745198) (end 94.22 52.28) (width 0.1524) (layer Back) (net 14))
+  (segment (start 94.22 52.28) (end 94.22 51.335) (width 0.1524) (layer Back) (net 14))
+  (via (at 89.00086 52.00076) (size 0.635) (layers Front Back) (net 14) (status 30))
+  (segment (start 89.00086 54.29924) (end 89.00086 52.00076) (width 0.1524) (layer Front) (net 14) (status 30))
+  (segment (start 94.22 51.335) (end 96.735 51.335) (width 0.1524) (layer Back) (net 14) (status 10))
+  (via (at 97.4 52) (size 0.635) (layers Front Back) (net 14) (status 30))
+  (segment (start 97.4 52) (end 97.4 51.99996) (width 0.1524) (layer Front) (net 14) (status 30))
+  (segment (start 97.4 51.99996) (end 97.35004 51.95) (width 0.1524) (layer Front) (net 14) (status 30))
+  (segment (start 96.735 51.335) (end 97.4 52) (width 0.1524) (layer Back) (net 14))
+  (segment (start 94.45 54.2) (end 96.7 54.2) (width 0.1524) (layer Front) (net 14) (status 30))
+  (segment (start 96.7 54.2) (end 96.85 54.05) (width 0.3048) (layer Front) (net 14) (status 30))
+  (segment (start 97.35004 51.95) (end 97.35004 52.59996) (width 0.1524) (layer Front) (net 14) (status 30))
+  (segment (start 96.85 53.1) (end 96.85 54.05) (width 0.1524) (layer Front) (net 14) (status 20))
+  (segment (start 97.35004 52.59996) (end 96.85 53.1) (width 0.1524) (layer Front) (net 14) (status 10))
+  (segment (start 97.35004 49.45) (end 97.35004 51.95) (width 0.1524) (layer Front) (net 14) (status 30))
+  (segment (start 97.2 51.79996) (end 97.35004 51.95) (width 0.3048) (layer Front) (net 14) (status 30))
   (zone (net 10) (net_name GNDPWR) (layer Front) (hatch edge 0.508)
     (connect_pads yes (clearance 0.25))
