File: Pot-timed/LED-strip_PWM__panel.kicad_pcb (KiCad board)
At the start: 2 copper layers, 99 x 100 mm, 14 parts

Commit message: Pot-timed (panel): filled with boards.
Parts:
- added C1: 100nF, MADW__C0805, F.Cu at (217.4, 155.2)
- added C1: 100nF, MADW__C0805, F.Cu at (195.4, 93.9)
- added C1: 100nF, MADW__C0805, F.Cu at (195.4, 124.5)
- added C1: 100nF, MADW__C0805, F.Cu at (195.4, 155.2)
- added C1: 100nF, MADW__C0805, F.Cu at (206.4, 155.2)
- added C1: 100nF, MADW__C0805, F.Cu at (206.4, 124.5)
- added C1: 100nF, MADW__C0805, F.Cu at (206.4, 93.9)
- added C1: 100nF, MADW__C0805, F.Cu at (184.4, 93.9)
- added C1: 100nF, MADW__C0805, F.Cu at (184.4, 124.5)
- added C1: 100nF, MADW__C0805, F.Cu at (184.4, 155.2)
- added C1: 100nF, MADW__C0805, F.Cu at (173.4, 155.2)
- added C1: 100nF, MADW__C0805, F.Cu at (217.4, 124.5)
- added C1: 100nF, MADW__C0805, F.Cu at (173.4, 124.5)
- added C1: 100nF, MADW__C0805, F.Cu at (173.4, 93.9)
- added C1: 100nF, MADW__C0805, F.Cu at (217.4, 93.9)
- added C1: 100nF, MADW__C0805, F.Cu at (239.4, 93.9)
- added C1: 100nF, MADW__C0805, F.Cu at (239.4, 124.5)
- added C1: 100nF, MADW__C0805, F.Cu at (239.4, 155.2)
- added C1: 100nF, MADW__C0805, F.Cu at (228.4, 155.2)
- added C1: 100nF, MADW__C0805, F.Cu at (228.4, 124.5)
- added C1: 100nF, MADW__C0805, F.Cu at (228.4, 93.9)
- added C2: 100nF, MADW__C0805, F.Cu at (223.4, 152.7)
- added C2: 100nF, MADW__C0805, F.Cu at (201.4, 91.4)
- added C2: 100nF, MADW__C0805, F.Cu at (201.4, 122.0)
- added C2: 100nF, MADW__C0805, F.Cu at (201.4, 152.7)
- added C2: 100nF, MADW__C0805, F.Cu at (212.4, 152.7)
- added C2: 100nF, MADW__C0805, F.Cu at (212.4, 122.0)
- added C2: 100nF, MADW__C0805, F.Cu at (212.4, 91.4)
- added C2: 100nF, MADW__C0805, F.Cu at (190.4, 91.4)
- added C2: 100nF, MADW__C0805, F.Cu at (190.4, 122.0)
- added C2: 100nF, MADW__C0805, F.Cu at (190.4, 152.7)
- added C2: 100nF, MADW__C0805, F.Cu at (179.4, 152.7)
- added C2: 100nF, MADW__C0805, F.Cu at (223.4, 122.0)
- added C2: 100nF, MADW__C0805, F.Cu at (179.4, 122.0)
- added C2: 100nF, MADW__C0805, F.Cu at (179.4, 91.4)
- added C2: 100nF, MADW__C0805, F.Cu at (223.4, 91.4)
- added C2: 100nF, MADW__C0805, F.Cu at (245.4, 91.4)
- added C2: 100nF, MADW__C0805, F.Cu at (245.4, 122.0)
- added C2: 100nF, MADW__C0805, F.Cu at (245.4, 152.7)
- added C2: 100nF, MADW__C0805, F.Cu at (234.4, 152.7)
- added C2: 100nF, MADW__C0805, F.Cu at (234.4, 122.0)
- added C2: 100nF, MADW__C0805, F.Cu at (234.4, 91.4)
- added C3: 4.7µF, MADW__C0805, F.Cu at (219.9, 155.2)
- added C3: 4.7µF, MADW__C0805, F.Cu at (197.9, 93.9)
- added C3: 4.7µF, MADW__C0805, F.Cu at (197.9, 124.5)
- added C3: 4.7µF, MADW__C0805, F.Cu at (197.9, 155.2)
- added C3: 4.7µF, MADW__C0805, F.Cu at (208.9, 155.2)
- added C3: 4.7µF, MADW__C0805, F.Cu at (208.9, 124.5)
- added C3: 4.7µF, MADW__C0805, F.Cu at (208.9, 93.9)
- added C3: 4.7µF, MADW__C0805, F.Cu at (186.9, 93.9)
- added C3: 4.7µF, MADW__C0805, F.Cu at (186.9, 124.5)
- added C3: 4.7µF, MADW__C0805, F.Cu at (186.9, 155.2)
- added C3: 4.7µF, MADW__C0805, F.Cu at (175.9, 155.2)
- added C3: 4.7µF, MADW__C0805, F.Cu at (219.9, 124.5)
- added C3: 4.7µF, MADW__C0805, F.Cu at (175.9, 124.5)
- added C3: 4.7µF, MADW__C0805, F.Cu at (175.9, 93.9)
- added C3: 4.7µF, MADW__C0805, F.Cu at (219.9, 93.9)
- added C3: 4.7µF, MADW__C0805, F.Cu at (241.9, 93.9)
- added C3: 4.7µF, MADW__C0805, F.Cu at (241.9, 124.5)
- added C3: 4.7µF, MADW__C0805, F.Cu at (241.9, 155.2)
- added C3: 4.7µF, MADW__C0805, F.Cu at (230.9, 155.2)
- added C3: 4.7µF, MADW__C0805, F.Cu at (230.9, 124.5)
- added C3: 4.7µF, MADW__C0805, F.Cu at (230.9, 93.9)
- added G1: OSHW-logo_silkscreen_3mm, OSHW-logo_silkscreen_3mm, B.Cu at (220.2, 168.0)
- added G1: OSHW-logo_silkscreen_3mm, OSHW-logo_silkscreen_3mm, B.Cu at (198.2, 106.7)
- added G1: OSHW-logo_silkscreen_3mm, OSHW-logo_silkscreen_3mm, B.Cu at (198.2, 137.4)
- added G1: OSHW-logo_silkscreen_3mm, OSHW-logo_silkscreen_3mm, B.Cu at (198.2, 168.0)
- added G1: OSHW-logo_silkscreen_3mm, OSHW-logo_silkscreen_3mm, B.Cu at (209.2, 168.0)
- added G1: OSHW-logo_silkscreen_3mm, OSHW-logo_silkscreen_3mm, B.Cu at (209.2, 137.4)
- added G1: OSHW-logo_silkscreen_3mm, OSHW-logo_silkscreen_3mm, B.Cu at (209.2, 106.7)
- added G1: OSHW-logo_silkscreen_3mm, OSHW-logo_silkscreen_3mm, B.Cu at (187.2, 106.7)
- added G1: OSHW-logo_silkscreen_3mm, OSHW-logo_silkscreen_3mm, B.Cu at (187.2, 137.4)
- added G1: OSHW-logo_silkscreen_3mm, OSHW-logo_silkscreen_3mm, B.Cu at (187.2, 168.0)
- added G1: OSHW-logo_silkscreen_3mm, OSHW-logo_silkscreen_3mm, B.Cu at (176.2, 168.0)
- added G1: OSHW-logo_silkscreen_3mm, OSHW-logo_silkscreen_3mm, B.Cu at (220.2, 137.4)
- added G1: OSHW-logo_silkscreen_3mm, OSHW-logo_silkscreen_3mm, B.Cu at (176.2, 137.4)
- added G1: OSHW-logo_silkscreen_3mm, OSHW-logo_silkscreen_3mm, B.Cu at (176.2, 106.7)
- added G1: OSHW-logo_silkscreen_3mm, OSHW-logo_silkscreen_3mm, B.Cu at (220.2, 106.7)
- added G1: OSHW-logo_silkscreen_3mm, OSHW-logo_silkscreen_3mm, B.Cu at (242.2, 106.7)
- added G1: OSHW-logo_silkscreen_3mm, OSHW-logo_silkscreen_3mm, B.Cu at (242.2, 137.4)
- added G1: OSHW-logo_silkscreen_3mm, OSHW-logo_silkscreen_3mm, B.Cu at (242.2, 168.0)
- added G1: OSHW-logo_silkscreen_3mm, OSHW-logo_silkscreen_3mm, B.Cu at (231.2, 168.0)
- added G1: OSHW-logo_silkscreen_3mm, OSHW-logo_silkscreen_3mm, B.Cu at (231.2, 137.4)
- added G1: OSHW-logo_silkscreen_3mm, OSHW-logo_silkscreen_3mm, B.Cu at (231.2, 106.7)
- added G2: LED_smile_silkscreen_3mm, LED_smile_silkscreen_3mm, B.Cu at (220.2, 157.0)
- added G2: LED_smile_silkscreen_3mm, LED_smile_silkscreen_3mm, B.Cu at (198.2, 95.7)
- added G2: LED_smile_silkscreen_3mm, LED_smile_silkscreen_3mm, B.Cu at (198.2, 126.3)
- added G2: LED_smile_silkscreen_3mm, LED_smile_silkscreen_3mm, B.Cu at (198.2, 157.0)
- added G2: LED_smile_silkscreen_3mm, LED_smile_silkscreen_3mm, B.Cu at (209.2, 157.0)
- added G2: LED_smile_silkscreen_3mm, LED_smile_silkscreen_3mm, B.Cu at (209.2, 126.3)
- added G2: LED_smile_silkscreen_3mm, LED_smile_silkscreen_3mm, B.Cu at (209.2, 95.7)
- added G2: LED_smile_silkscreen_3mm, LED_smile_silkscreen_3mm, B.Cu at (187.2, 95.7)
- added G2: LED_smile_silkscreen_3mm, LED_smile_silkscreen_3mm, B.Cu at (187.2, 126.3)
- added G2: LED_smile_silkscreen_3mm, LED_smile_silkscreen_3mm, B.Cu at (187.2, 157.0)
- added G2: LED_smile_silkscreen_3mm, LED_smile_silkscreen_3mm, B.Cu at (176.2, 157.0)
- added G2: LED_smile_silkscreen_3mm, LED_smile_silkscreen_3mm, B.Cu at (220.2, 126.3)
- added G2: LED_smile_silkscreen_3mm, LED_smile_silkscreen_3mm, B.Cu at (176.2, 126.3)
- added G2: LED_smile_silkscreen_3mm, LED_smile_silkscreen_3mm, B.Cu at (176.2, 95.7)
- added G2: LED_smile_silkscreen_3mm, LED_smile_silkscreen_3mm, B.Cu at (220.2, 95.7)
- added G2: LED_smile_silkscreen_3mm, LED_smile_silkscreen_3mm, B.Cu at (242.2, 95.7)
- added G2: LED_smile_silkscreen_3mm, LED_smile_silkscreen_3mm, B.Cu at (242.2, 126.3)
- added G2: LED_smile_silkscreen_3mm, LED_smile_silkscreen_3mm, B.Cu at (242.2, 157.0)
- added G2: LED_smile_silkscreen_3mm, LED_smile_silkscreen_3mm, B.Cu at (231.2, 157.0)
- added G2: LED_smile_silkscreen_3mm, LED_smile_silkscreen_3mm, B.Cu at (231.2, 126.3)
- added G2: LED_smile_silkscreen_3mm, LED_smile_silkscreen_3mm, B.Cu at (231.2, 95.7)
- added IC1: MADW__ATTINY13-MM, MADW__MLF10, F.Cu at (223.2, 160.5)
- added IC1: MADW__ATTINY13-MM, MADW__MLF10, F.Cu at (201.2, 99.2)
- added IC1: MADW__ATTINY13-MM, MADW__MLF10, F.Cu at (201.2, 129.9)
- added IC1: MADW__ATTINY13-MM, MADW__MLF10, F.Cu at (201.2, 160.5)
- added IC1: MADW__ATTINY13-MM, MADW__MLF10, F.Cu at (212.2, 160.5)
- added IC1: MADW__ATTINY13-MM, MADW__MLF10, F.Cu at (212.2, 129.9)
- added IC1: MADW__ATTINY13-MM, MADW__MLF10, F.Cu at (212.2, 99.2)
- added IC1: MADW__ATTINY13-MM, MADW__MLF10, F.Cu at (190.2, 99.2)
- added IC1: MADW__ATTINY13-MM, MADW__MLF10, F.Cu at (190.2, 129.9)
- added IC1: MADW__ATTINY13-MM, MADW__MLF10, F.Cu at (190.2, 160.5)
- added IC1: MADW__ATTINY13-MM, MADW__MLF10, F.Cu at (179.2, 160.5)
- added IC1: MADW__ATTINY13-MM, MADW__MLF10, F.Cu at (223.2, 129.9)
- added IC1: MADW__ATTINY13-MM, MADW__MLF10, F.Cu at (179.2, 129.9)
- added IC1: MADW__ATTINY13-MM, MADW__MLF10, F.Cu at (179.2, 99.2)
- added IC1: MADW__ATTINY13-MM, MADW__MLF10, F.Cu at (223.2, 99.2)
- added IC1: MADW__ATTINY13-MM, MADW__MLF10, F.Cu at (245.2, 99.2)
- added IC1: MADW__ATTINY13-MM, MADW__MLF10, F.Cu at (245.2, 129.9)
- added IC1: MADW__ATTINY13-MM, MADW__MLF10, F.Cu at (245.2, 160.5)
- added IC1: MADW__ATTINY13-MM, MADW__MLF10, F.Cu at (234.2, 160.5)
- added IC1: MADW__ATTINY13-MM, MADW__MLF10, F.Cu at (234.2, 129.9)
- added IC1: MADW__ATTINY13-MM, MADW__MLF10, F.Cu at (234.2, 99.2)
- added JP1: ISP, MADW__PIN_ARRAY_3x2_1.27mm, F.Cu at (218.7, 160.5)
- added JP1: ISP, MADW__PIN_ARRAY_3x2_1.27mm, F.Cu at (196.7, 99.2)
- added JP1: ISP, MADW__PIN_ARRAY_3x2_1.27mm, F.Cu at (196.7, 129.9)
- added JP1: ISP, MADW__PIN_ARRAY_3x2_1.27mm, F.Cu at (196.7, 160.5)
- added JP1: ISP, MADW__PIN_ARRAY_3x2_1.27mm, F.Cu at (207.7, 160.5)
- added JP1: ISP, MADW__PIN_ARRAY_3x2_1.27mm, F.Cu at (207.7, 129.9)
- added JP1: ISP, MADW__PIN_ARRAY_3x2_1.27mm, F.Cu at (207.7, 99.2)
- added JP1: ISP, MADW__PIN_ARRAY_3x2_1.27mm, F.Cu at (185.7, 99.2)
- added JP1: ISP, MADW__PIN_ARRAY_3x2_1.27mm, F.Cu at (185.7, 129.9)
- added JP1: ISP, MADW__PIN_ARRAY_3x2_1.27mm, F.Cu at (185.7, 160.5)
- added JP1: ISP, MADW__PIN_ARRAY_3x2_1.27mm, F.Cu at (174.7, 160.5)
- added JP1: ISP, MADW__PIN_ARRAY_3x2_1.27mm, F.Cu at (218.7, 129.9)
- added JP1: ISP, MADW__PIN_ARRAY_3x2_1.27mm, F.Cu at (174.7, 129.9)
- added JP1: ISP, MADW__PIN_ARRAY_3x2_1.27mm, F.Cu at (174.7, 99.2)
- added JP1: ISP, MADW__PIN_ARRAY_3x2_1.27mm, F.Cu at (218.7, 99.2)
- added JP1: ISP, MADW__PIN_ARRAY_3x2_1.27mm, F.Cu at (240.7, 99.2)
- added JP1: ISP, MADW__PIN_ARRAY_3x2_1.27mm, F.Cu at (240.7, 129.9)
- added JP1: ISP, MADW__PIN_ARRAY_3x2_1.27mm, F.Cu at (240.7, 160.5)
- added JP1: ISP, MADW__PIN_ARRAY_3x2_1.27mm, F.Cu at (229.7, 160.5)
- added JP1: ISP, MADW__PIN_ARRAY_3x2_1.27mm, F.Cu at (229.7, 129.9)
- added JP1: ISP, MADW__PIN_ARRAY_3x2_1.27mm, F.Cu at (229.7, 99.2)
- added NJ1: NET-JOIN, MADW__SMD-net-noin-0.5mm, F.Cu at (219.9, 152.1)
- added NJ1: NET-JOIN, MADW__SMD-net-noin-0.5mm, F.Cu at (197.9, 90.8)
- added NJ1: NET-JOIN, MADW__SMD-net-noin-0.5mm, F.Cu at (197.9, 121.5)
- added NJ1: NET-JOIN, MADW__SMD-net-noin-0.5mm, F.Cu at (197.9, 152.1)
- added NJ1: NET-JOIN, MADW__SMD-net-noin-0.5mm, F.Cu at (208.9, 152.1)
- added NJ1: NET-JOIN, MADW__SMD-net-noin-0.5mm, F.Cu at (208.9, 121.5)
- added NJ1: NET-JOIN, MADW__SMD-net-noin-0.5mm, F.Cu at (208.9, 90.8)
- added NJ1: NET-JOIN, MADW__SMD-net-noin-0.5mm, F.Cu at (186.9, 90.8)
- added NJ1: NET-JOIN, MADW__SMD-net-noin-0.5mm, F.Cu at (186.9, 121.5)
- added NJ1: NET-JOIN, MADW__SMD-net-noin-0.5mm, F.Cu at (186.9, 152.1)
- added NJ1: NET-JOIN, MADW__SMD-net-noin-0.5mm, F.Cu at (175.9, 152.1)
- added NJ1: NET-JOIN, MADW__SMD-net-noin-0.5mm, F.Cu at (219.9, 121.5)
- added NJ1: NET-JOIN, MADW__SMD-net-noin-0.5mm, F.Cu at (175.9, 121.5)
- added NJ1: NET-JOIN, MADW__SMD-net-noin-0.5mm, F.Cu at (175.9, 90.8)
- added NJ1: NET-JOIN, MADW__SMD-net-noin-0.5mm, F.Cu at (219.9, 90.8)
- added NJ1: NET-JOIN, MADW__SMD-net-noin-0.5mm, F.Cu at (241.9, 90.8)
- added NJ1: NET-JOIN, MADW__SMD-net-noin-0.5mm, F.Cu at (241.9, 121.5)
- added NJ1: NET-JOIN, MADW__SMD-net-noin-0.5mm, F.Cu at (241.9, 152.1)
- added NJ1: NET-JOIN, MADW__SMD-net-noin-0.5mm, F.Cu at (230.9, 152.1)
- added NJ1: NET-JOIN, MADW__SMD-net-noin-0.5mm, F.Cu at (230.9, 121.5)
- added NJ1: NET-JOIN, MADW__SMD-net-noin-0.5mm, F.Cu at (230.9, 90.8)
- added P1: CONN_2, MADW__SIL-2, F.Cu at (221.0, 149.6)
- added P1: CONN_2, MADW__SIL-2, F.Cu at (199.0, 88.3)
- added P1: CONN_2, MADW__SIL-2, F.Cu at (199.0, 118.9)
- added P1: CONN_2, MADW__SIL-2, F.Cu at (199.0, 149.6)
- added P1: CONN_2, MADW__SIL-2, F.Cu at (210.0, 149.6)
- added P1: CONN_2, MADW__SIL-2, F.Cu at (210.0, 118.9)
- added P1: CONN_2, MADW__SIL-2, F.Cu at (210.0, 88.3)
- added P1: CONN_2, MADW__SIL-2, F.Cu at (188.0, 88.3)
- added P1: CONN_2, MADW__SIL-2, F.Cu at (188.0, 118.9)
- added P1: CONN_2, MADW__SIL-2, F.Cu at (188.0, 149.6)
- added P1: CONN_2, MADW__SIL-2, F.Cu at (177.0, 149.6)
- added P1: CONN_2, MADW__SIL-2, F.Cu at (221.0, 118.9)
- added P1: CONN_2, MADW__SIL-2, F.Cu at (177.0, 118.9)
- added P1: CONN_2, MADW__SIL-2, F.Cu at (177.0, 88.3)
- added P1: CONN_2, MADW__SIL-2, F.Cu at (221.0, 88.3)
- added P1: CONN_2, MADW__SIL-2, F.Cu at (243.0, 88.3)
- added P1: CONN_2, MADW__SIL-2, F.Cu at (243.0, 118.9)
- added P1: CONN_2, MADW__SIL-2, F.Cu at (243.0, 149.6)
- added P1: CONN_2, MADW__SIL-2, F.Cu at (232.0, 149.6)
- added P1: CONN_2, MADW__SIL-2, F.Cu at (232.0, 118.9)
- added P1: CONN_2, MADW__SIL-2, F.Cu at (232.0, 88.3)
- added P2: CONN_2, MADW__SIL-2, F.Cu at (221.0, 175.8)
- added P2: CONN_2, MADW__SIL-2, F.Cu at (199.0, 114.5)
- added P2: CONN_2, MADW__SIL-2, F.Cu at (199.0, 145.1)
- added P2: CONN_2, MADW__SIL-2, F.Cu at (199.0, 175.8)
- added P2: CONN_2, MADW__SIL-2, F.Cu at (210.0, 175.8)
- added P2: CONN_2, MADW__SIL-2, F.Cu at (210.0, 145.1)
- added P2: CONN_2, MADW__SIL-2, F.Cu at (210.0, 114.5)
- added P2: CONN_2, MADW__SIL-2, F.Cu at (188.0, 114.5)
- added P2: CONN_2, MADW__SIL-2, F.Cu at (188.0, 145.1)
- added P2: CONN_2, MADW__SIL-2, F.Cu at (188.0, 175.8)
- added P2: CONN_2, MADW__SIL-2, F.Cu at (177.0, 175.8)
- added P2: CONN_2, MADW__SIL-2, F.Cu at (221.0, 145.1)
- added P2: CONN_2, MADW__SIL-2, F.Cu at (177.0, 145.1)
- added P2: CONN_2, MADW__SIL-2, F.Cu at (177.0, 114.5)
- added P2: CONN_2, MADW__SIL-2, F.Cu at (221.0, 114.5)
- added P2: CONN_2, MADW__SIL-2, F.Cu at (243.0, 114.5)
- added P2: CONN_2, MADW__SIL-2, F.Cu at (243.0, 145.1)
- added P2: CONN_2, MADW__SIL-2, F.Cu at (243.0, 175.8)
- added P2: CONN_2, MADW__SIL-2, F.Cu at (232.0, 175.8)
- added P2: CONN_2, MADW__SIL-2, F.Cu at (232.0, 145.1)
- added P2: CONN_2, MADW__SIL-2, F.Cu at (232.0, 114.5)
- added R1: 100k, MADW__R0603_2, F.Cu at (217.8, 171.7)
- added R1: 100k, MADW__R0603_2, F.Cu at (195.8, 110.4)
- added R1: 100k, MADW__R0603_2, F.Cu at (195.8, 141.0)
- added R1: 100k, MADW__R0603_2, F.Cu at (195.8, 171.7)
- added R1: 100k, MADW__R0603_2, F.Cu at (206.8, 171.7)
- added R1: 100k, MADW__R0603_2, F.Cu at (206.8, 141.0)
- added R1: 100k, MADW__R0603_2, F.Cu at (206.8, 110.4)
- added R1: 100k, MADW__R0603_2, F.Cu at (184.8, 110.4)
- added R1: 100k, MADW__R0603_2, F.Cu at (184.8, 141.0)
- added R1: 100k, MADW__R0603_2, F.Cu at (184.8, 171.7)
- added R1: 100k, MADW__R0603_2, F.Cu at (173.8, 171.7)
- added R1: 100k, MADW__R0603_2, F.Cu at (217.8, 141.0)
- added R1: 100k, MADW__R0603_2, F.Cu at (173.8, 141.0)
- added R1: 100k, MADW__R0603_2, F.Cu at (173.8, 110.4)
- added R1: 100k, MADW__R0603_2, F.Cu at (217.8, 110.4)
- added R1: 100k, MADW__R0603_2, F.Cu at (239.8, 110.4)
- added R1: 100k, MADW__R0603_2, F.Cu at (239.8, 141.0)
- added R1: 100k, MADW__R0603_2, F.Cu at (239.8, 171.7)
- added R1: 100k, MADW__R0603_2, F.Cu at (228.8, 171.7)
- added R1: 100k, MADW__R0603_2, F.Cu at (228.8, 141.0)
- added R1: 100k, MADW__R0603_2, F.Cu at (228.8, 110.4)
- added R2: 150R, MADW__R0603_2, F.Cu at (224.2, 171.6)
- added R2: 150R, MADW__R0603_2, F.Cu at (202.2, 110.3)
- added R2: 150R, MADW__R0603_2, F.Cu at (202.2, 140.9)
- added R2: 150R, MADW__R0603_2, F.Cu at (202.2, 171.6)
- added R2: 150R, MADW__R0603_2, F.Cu at (213.2, 171.6)
- added R2: 150R, MADW__R0603_2, F.Cu at (213.2, 140.9)
- added R2: 150R, MADW__R0603_2, F.Cu at (213.2, 110.3)
- added R2: 150R, MADW__R0603_2, F.Cu at (191.2, 110.3)
- added R2: 150R, MADW__R0603_2, F.Cu at (191.2, 140.9)
- added R2: 150R, MADW__R0603_2, F.Cu at (191.2, 171.6)
- added R2: 150R, MADW__R0603_2, F.Cu at (180.2, 171.6)
- added R2: 150R, MADW__R0603_2, F.Cu at (224.2, 140.9)
- added R2: 150R, MADW__R0603_2, F.Cu at (180.2, 140.9)
- added R2: 150R, MADW__R0603_2, F.Cu at (180.2, 110.3)
- added R2: 150R, MADW__R0603_2, F.Cu at (224.2, 110.3)
- added R2: 150R, MADW__R0603_2, F.Cu at (246.2, 110.3)
- added R2: 150R, MADW__R0603_2, F.Cu at (246.2, 140.9)
- added R2: 150R, MADW__R0603_2, F.Cu at (246.2, 171.6)
- added R2: 150R, MADW__R0603_2, F.Cu at (235.2, 171.6)
- added R2: 150R, MADW__R0603_2, F.Cu at (235.2, 140.9)
- added R2: 150R, MADW__R0603_2, F.Cu at (235.2, 110.3)
- added RV1: 50k, MADW__TC33X-POT, F.Cu at (219.1, 166.3)
- added RV1: 50k, MADW__TC33X-POT, F.Cu at (197.1, 105.0)
- added RV1: 50k, MADW__TC33X-POT, F.Cu at (197.1, 135.7)
- added RV1: 50k, MADW__TC33X-POT, F.Cu at (197.1, 166.3)
- added RV1: 50k, MADW__TC33X-POT, F.Cu at (208.1, 166.3)
- added RV1: 50k, MADW__TC33X-POT, F.Cu at (208.1, 135.7)
- added RV1: 50k, MADW__TC33X-POT, F.Cu at (208.1, 105.0)
- added RV1: 50k, MADW__TC33X-POT, F.Cu at (186.1, 105.0)
- added RV1: 50k, MADW__TC33X-POT, F.Cu at (186.1, 135.7)
- added RV1: 50k, MADW__TC33X-POT, F.Cu at (186.1, 166.3)
- added RV1: 50k, MADW__TC33X-POT, F.Cu at (175.1, 166.3)
- added RV1: 50k, MADW__TC33X-POT, F.Cu at (219.1, 135.7)
- added RV1: 50k, MADW__TC33X-POT, F.Cu at (175.1, 135.7)
- added RV1: 50k, MADW__TC33X-POT, F.Cu at (175.1, 105.0)
- added RV1: 50k, MADW__TC33X-POT, F.Cu at (219.1, 105.0)
- added RV1: 50k, MADW__TC33X-POT, F.Cu at (241.1, 105.0)
- added RV1: 50k, MADW__TC33X-POT, F.Cu at (241.1, 135.7)
- added RV1: 50k, MADW__TC33X-POT, F.Cu at (241.1, 166.3)
- added RV1: 50k, MADW__TC33X-POT, F.Cu at (230.1, 166.3)
- added RV1: 50k, MADW__TC33X-POT, F.Cu at (230.1, 135.7)
- added RV1: 50k, MADW__TC33X-POT, F.Cu at (230.1, 105.0)
- added RV2: 50k, MADW__TC33X-POT, F.Cu at (223.1, 166.3)
- added RV2: 50k, MADW__TC33X-POT, F.Cu at (201.1, 105.0)
- added RV2: 50k, MADW__TC33X-POT, F.Cu at (201.1, 135.7)
- added RV2: 50k, MADW__TC33X-POT, F.Cu at (201.1, 166.3)
- added RV2: 50k, MADW__TC33X-POT, F.Cu at (212.1, 166.3)
- added RV2: 50k, MADW__TC33X-POT, F.Cu at (212.1, 135.7)
- added RV2: 50k, MADW__TC33X-POT, F.Cu at (212.1, 105.0)
- added RV2: 50k, MADW__TC33X-POT, F.Cu at (190.1, 105.0)
- added RV2: 50k, MADW__TC33X-POT, F.Cu at (190.1, 135.7)
- added RV2: 50k, MADW__TC33X-POT, F.Cu at (190.1, 166.3)
- added RV2: 50k, MADW__TC33X-POT, F.Cu at (179.1, 166.3)
- added RV2: 50k, MADW__TC33X-POT, F.Cu at (223.1, 135.7)
- added RV2: 50k, MADW__TC33X-POT, F.Cu at (179.1, 135.7)
- added RV2: 50k, MADW__TC33X-POT, F.Cu at (179.1, 105.0)
- added RV2: 50k, MADW__TC33X-POT, F.Cu at (223.1, 105.0)
- added RV2: 50k, MADW__TC33X-POT, F.Cu at (245.1, 105.0)
- added RV2: 50k, MADW__TC33X-POT, F.Cu at (245.1, 135.7)
- added RV2: 50k, MADW__TC33X-POT, F.Cu at (245.1, 166.3)
- added RV2: 50k, MADW__TC33X-POT, F.Cu at (234.1, 166.3)
- added RV2: 50k, MADW__TC33X-POT, F.Cu at (234.1, 135.7)
- added RV2: 50k, MADW__TC33X-POT, F.Cu at (234.1, 105.0)
- added T1: AO3400, MADW__SOT23, F.Cu at (221.0, 171.6)
- added T1: AO3400, MADW__SOT23, F.Cu at (199.0, 110.3)
- added T1: AO3400, MADW__SOT23, F.Cu at (199.0, 140.9)
- added T1: AO3400, MADW__SOT23, F.Cu at (199.0, 171.6)
- added T1: AO3400, MADW__SOT23, F.Cu at (210.0, 171.6)
- added T1: AO3400, MADW__SOT23, F.Cu at (210.0, 140.9)
- added T1: AO3400, MADW__SOT23, F.Cu at (210.0, 110.3)
- added T1: AO3400, MADW__SOT23, F.Cu at (188.0, 110.3)
- added T1: AO3400, MADW__SOT23, F.Cu at (188.0, 140.9)
- added T1: AO3400, MADW__SOT23, F.Cu at (188.0, 171.6)
- added T1: AO3400, MADW__SOT23, F.Cu at (177.0, 171.6)
- added T1: AO3400, MADW__SOT23, F.Cu at (221.0, 140.9)
- added T1: AO3400, MADW__SOT23, F.Cu at (177.0, 140.9)
- added T1: AO3400, MADW__SOT23, F.Cu at (177.0, 110.3)
- added T1: AO3400, MADW__SOT23, F.Cu at (221.0, 110.3)
- added T1: AO3400, MADW__SOT23, F.Cu at (243.0, 110.3)
- added T1: AO3400, MADW__SOT23, F.Cu at (243.0, 140.9)
- added T1: AO3400, MADW__SOT23, F.Cu at (243.0, 171.6)
- added T1: AO3400, MADW__SOT23, F.Cu at (232.0, 171.6)
- added T1: AO3400, MADW__SOT23, F.Cu at (232.0, 140.9)
- added T1: AO3400, MADW__SOT23, F.Cu at (232.0, 110.3)
- added U1: MCP1804-SOT23-5, MADW__SOT23-5, F.Cu at (223.3, 155.7)
- added U1: MCP1804-SOT23-5, MADW__SOT23-5, F.Cu at (201.3, 94.4)
- added U1: MCP1804-SOT23-5, MADW__SOT23-5, F.Cu at (201.3, 125.0)
- added U1: MCP1804-SOT23-5, MADW__SOT23-5, F.Cu at (201.3, 155.7)
- added U1: MCP1804-SOT23-5, MADW__SOT23-5, F.Cu at (212.3, 155.7)
- added U1: MCP1804-SOT23-5, MADW__SOT23-5, F.Cu at (212.3, 125.0)
- added U1: MCP1804-SOT23-5, MADW__SOT23-5, F.Cu at (212.3, 94.4)
- added U1: MCP1804-SOT23-5, MADW__SOT23-5, F.Cu at (190.3, 94.4)
- added U1: MCP1804-SOT23-5, MADW__SOT23-5, F.Cu at (190.3, 125.0)
- added U1: MCP1804-SOT23-5, MADW__SOT23-5, F.Cu at (190.3, 155.7)
- added U1: MCP1804-SOT23-5, MADW__SOT23-5, F.Cu at (179.3, 155.7)
- added U1: MCP1804-SOT23-5, MADW__SOT23-5, F.Cu at (223.3, 125.0)
- added U1: MCP1804-SOT23-5, MADW__SOT23-5, F.Cu at (179.3, 125.0)
- added U1: MCP1804-SOT23-5, MADW__SOT23-5, F.Cu at (179.3, 94.4)
- added U1: MCP1804-SOT23-5, MADW__SOT23-5, F.Cu at (223.3, 94.4)
- added U1: MCP1804-SOT23-5, MADW__SOT23-5, F.Cu at (245.3, 94.4)
- added U1: MCP1804-SOT23-5, MADW__SOT23-5, F.Cu at (245.3, 125.0)
- added U1: MCP1804-SOT23-5, MADW__SOT23-5, F.Cu at (245.3, 155.7)
- added U1: MCP1804-SOT23-5, MADW__SOT23-5, F.Cu at (234.3, 155.7)
- added U1: MCP1804-SOT23-5, MADW__SOT23-5, F.Cu at (234.3, 125.0)
- added U1: MCP1804-SOT23-5, MADW__SOT23-5, F.Cu at (234.3, 94.4)
Routing:
- net GNDPWR: track 0.00 -> 884.9 mm, vias 0 -> 105
- net /Vin: track 0.00 -> 797.8 mm, vias 0 -> 21
- net GND: track 0.00 -> 725.5 mm, vias 0 -> 42
- net /MOSI: track 0.00 -> 637.8 mm
- net VCC: track 0.00 -> 430.9 mm, vias 0 -> 42
- net /POT1: track 0.00 -> 297.1 mm
- net /SCK: track 0.00 -> 245.7 mm
- net /POT2: track 0.00 -> 205.6 mm
- net /MISO: track 0.00 -> 183.6 mm
- net /RESET: track 0.00 -> 126.4 mm
- net /drain: track 0.00 -> 89.1 mm
- net N-000004: track 0.00 -> 56.9 mm
- added copper zone on F.Cu, net GND
- added copper zone on B.Cu, net GNDPWR
- added copper zone on F.Cu, net GNDPWR
Other:
- net class Default: via_dia 0.635 -> 0.762
- net class Power: via_dia 0.635 -> 0.762
- rule via_min_drill: 0.3302 -> 0.3
- rule via_min_size: 0.635 -> 0.6
- board text added: "+"
- board text added: "-"
- board text added: "12V"
- board text added: "2013 - blog.spitzenpfeil.org"
- board text added: "LED"
- board text added: "V0.12 POT PWM controller"

Commit message: Pot-timed (s.b.): added alternative MOSFET to schematic + Rev. update.
Other:
- board text added: "V0.12.a POT PWM controller"
- board text removed: "V0.12 POT PWM controller"
Changed lines of the file:
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@@
     (effects (font (size 1 1) (thickness 0.2032)) (justify mirror))
   )
-  (gr_text "V0.12\nPOT PWM controller" (at 221.2 162.475 90) (layer B.SilkS)
+  (gr_text "V0.12.a\nPOT PWM controller" (at 221.2 162.475 90) (layer B.SilkS)
     (effects (font (size 1 1) (thickness 0.2032)) (justify mirror))
   )
@@
     (effects (font (size 1 1) (thickness 0.2032)) (justify mirror))
   )
-  (gr_text "V0.12\nPOT PWM controller" (at 221.2 131.825 90) (layer B.SilkS)
+  (gr_text "V0.12.a\nPOT PWM controller" (at 221.2 131.825 90) (layer B.SilkS)
     (effects (font (size 1 1) (thickness 0.2032)) (justify mirror))
   )
@@
     (effects (font (size 1 1) (thickness 0.2032)) (justify mirror))
   )
-  (gr_text "V0.12\nPOT PWM controller" (at 221.2 101.175 90) (layer B.SilkS)
+  (gr_text "V0.12.a\nPOT PWM controller" (at 221.2 101.175 90) (layer B.SilkS)
     (effects (font (size 1 1) (thickness 0.2032)) (justify mirror))
   )
@@
     (effects (font (size 1 1) (thickness 0.2)) (justify mirror))
   )
-  (gr_text "V0.12\nPOT PWM controller" (at 243.2 101.175 90) (layer B.SilkS)
+  (gr_text "V0.12.a\nPOT PWM controller" (at 243.2 101.175 90) (layer B.SilkS)
     (effects (font (size 1 1) (thickness 0.2032)) (justify mirror))
   )
@@
     (effects (font (size 1 1) (thickness 0.2)) (justify mirror))
   )
-  (gr_text "V0.12\nPOT PWM controller" (at 243.2 131.825 90) (layer B.SilkS)
+  (gr_text "V0.12.a\nPOT PWM controller" (at 243.2 131.825 90) (layer B.SilkS)
     (effects (font (size 1 1) (thickness 0.2032)) (justify mirror))
   )
@@
     (effects (font (size 1 1) (thickness 0.2)) (justify mirror))
   )
-  (gr_text "V0.12\nPOT PWM controller" (at 243.2 162.475 90) (layer B.SilkS)
+  (gr_text "V0.12.a\nPOT PWM controller" (at 243.2 162.475 90) (layer B.SilkS)
     (effects (font (size 1 1) (thickness 0.2032)) (justify mirror))
   )
@@
     (effects (font (size 1 1) (thickness 0.2032)) (justify mirror))
   )
-  (gr_text "V0.12\nPOT PWM controller" (at 232.2 162.475 90) (layer B.SilkS)
+  (gr_text "V0.12.a\nPOT PWM controller" (at 232.2 162.475 90) (layer B.SilkS)
     (effects (font (size 1 1) (thickness 0.2032)) (justify mirror))
   )
@@
     (effects (font (size 1 1) (thickness 0.2032)) (justify mirror))
   )
-  (gr_text "V0.12\nPOT PWM controller" (at 232.2 131.825 90) (layer B.SilkS)
+  (gr_text "V0.12.a\nPOT PWM controller" (at 232.2 131.825 90) (layer B.SilkS)
     (effects (font (size 1 1) (thickness 0.2032)) (justify mirror))
   )
@@
     (effects (font (size 1 1) (thickness 0.2032)) (justify mirror))
   )
-  (gr_text "V0.12\nPOT PWM controller" (at 232.2 101.175 90) (layer B.SilkS)
+  (gr_text "V0.12.a\nPOT PWM controller" (at 232.2 101.175 90) (layer B.SilkS)
     (effects (font (size 1 1) (thickness 0.2032)) (justify mirror))
   )
@@
     (effects (font (size 1 1) (thickness 0.2)) (justify mirror))
   )
-  (gr_text "V0.12\nPOT PWM controller" (at 199.2 101.175 90) (layer B.SilkS)
+  (gr_text "V0.12.a\nPOT PWM controller" (at 199.2 101.175 90) (layer B.SilkS)
     (effects (font (size 1 1) (thickness 0.2032)) (justify mirror))
   )
@@
     (effects (font (size 1 1) (thickness 0.2)) (justify mirror))
   )
-  (gr_text "V0.12\nPOT PWM controller" (at 199.2 131.825 90) (layer B.SilkS)
+  (gr_text "V0.12.a\nPOT PWM controller" (at 199.2 131.825 90) (layer B.SilkS)
     (effects (font (size 1 1) (thickness 0.2032)) (justify mirror))
   )
@@
     (effects (font (size 1 1) (thickness 0.2)) (justify mirror))
   )
-  (gr_text "V0.12\nPOT PWM controller" (at 199.2 162.475 90) (layer B.SilkS)
+  (gr_text "V0.12.a\nPOT PWM controller" (at 199.2 162.475 90) (layer B.SilkS)
     (effects (font (size 1 1) (thickness 0.2032)) (justify mirror))
   )
@@
     (effects (font (size 1 1) (thickness 0.2032)) (justify mirror))
   )
-  (gr_text "V0.12\nPOT PWM controller" (at 210.2 162.475 90) (layer B.SilkS)
+  (gr_text "V0.12.a\nPOT PWM controller" (at 210.2 162.475 90) (layer B.SilkS)
     (effects (font (size 1 1) (thickness 0.2032)) (justify mirror))
   )
@@
     (effects (font (size 1 1) (thickness 0.2032)) (justify mirror))
   )
-  (gr_text "V0.12\nPOT PWM controller" (at 210.2 131.825 90) (layer B.SilkS)
+  (gr_text "V0.12.a\nPOT PWM controller" (at 210.2 131.825 90) (layer B.SilkS)
     (effects (font (size 1 1) (thickness 0.2032)) (justify mirror))
   )
@@
     (effects (font (size 1 1) (thickness 0.2032)) (justify mirror))
   )
-  (gr_text "V0.12\nPOT PWM controller" (at 210.2 101.175 90) (layer B.SilkS)
+  (gr_text "V0.12.a\nPOT PWM controller" (at 210.2 101.175 90) (layer B.SilkS)
     (effects (font (size 1 1) (thickness 0.2032)) (justify mirror))
   )
@@
     (effects (font (size 1 1) (thickness 0.2)) (justify mirror))
   )
-  (gr_text "V0.12\nPOT PWM controller" (at 188.2 101.175 90) (layer B.SilkS)
+  (gr_text "V0.12.a\nPOT PWM controller" (at 188.2 101.175 90) (layer B.SilkS)
     (effects (font (size 1 1) (thickness 0.2032)) (justify mirror))
   )
@@
     (effects (font (size 1 1) (thickness 0.2)) (justify mirror))
   )
-  (gr_text "V0.12\nPOT PWM controller" (at 188.2 131.825 90) (layer B.SilkS)
+  (gr_text "V0.12.a\nPOT PWM controller" (at 188.2 131.825 90) (layer B.SilkS)
     (effects (font (size 1 1) (thickness 0.2032)) (justify mirror))
   )
@@
     (effects (font (size 1 1) (thickness 0.2)) (justify mirror))
   )
-  (gr_text "V0.12\nPOT PWM controller" (at 188.2 162.475 90) (layer B.SilkS)
+  (gr_text "V0.12.a\nPOT PWM controller" (at 188.2 162.475 90) (layer B.SilkS)
     (effects (font (size 1 1) (thickness 0.2032)) (justify mirror))
   )
@@
     (effects (font (size 1 1) (thickness 0.2032)) (justify mirror))
   )
-  (gr_text "V0.12\nPOT PWM controller" (at 177.2 162.475 90) (layer B.SilkS)
+  (gr_text "V0.12.a\nPOT PWM controller" (at 177.2 162.475 90) (layer B.SilkS)
     (effects (font (size 1 1) (thickness 0.2032)) (justify mirror))
   )
@@
     (effects (font (size 1 1) (thickness 0.2032)) (justify mirror))
   )
-  (gr_text "V0.12\nPOT PWM controller" (at 177.2 131.825 90) (layer B.SilkS)
+  (gr_text "V0.12.a\nPOT PWM controller" (at 177.2 131.825 90) (layer B.SilkS)
     (effects (font (size 1 1) (thickness 0.2032)) (justify mirror))
   )
@@
     (effects (font (size 1 1) (thickness 0.2032)) (justify mirror))
   )
-  (gr_text "V0.12\nPOT PWM controller" (at 177.2 101.175 90) (layer B.SilkS)
-    (effects (font (size 1 1) (thickness 0.2032)) (justify mirror))
-  )
+  (gr_text "V0.12.a\nPOT PWM controller" (at 177.2 101.175 90) (layer B.SilkS)
+    (effects (font (size 1 1) (thickness 0.2032)) (justify mirror))
+  )
