File: Switch-timed/LED-strip_PWM.kicad_pcb (KiCad board)
At the start: 2 copper layers, 32 x 16 mm, 15 parts, among them IC1 ATTINY13A-MM, P1 CONN_2, P2 CONN_2, T1 AO3400, U1 MCP6001, U2 MCP1804-SOT23-5

Commit message: Changed to custom attiny13 schematic symbol + footprint.
Parts:
- added DS1: BAT54, MADW__SOT23, F.Cu at (99.2, 65.2)
- added R4: 500k, MADW__R0603_2, F.Cu at (93.3, 67.0)
- IC1: value ATTINY13A-MM -> MADW__ATTINY13-MM
Connections:
- IC1 pad 3: (no net) -> N-000006
- IC1 pad 8: (no net) -> N-000007
Changed lines of the file:
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@@
-(kicad_pcb (version 3) (host pcbnew "(2013-05-24 BZR 4164)-testing")
+(kicad_pcb (version 3) (host pcbnew "(2013-06-07 BZR 4197)-testing")
   (general
-    (links 32)
-    (no_connects 31)
-    (area 51.494973 41.849999 108.100001 60.2332)
+    (links 37)
+    (no_connects 36)
+    (area 51.494973 41.849999 108.100001 69.9532)
     (thickness 1.6002)
     (drawings 6)
     (tracks 8)
     (zones 0)
-    (modules 15)
-    (nets 15)
+    (modules 17)
+    (nets 17)
   )
   (page User 431.8 279.4)
@@
   (net 9 GND)
   (net 10 GNDPWR)
-  (net 11 N-000001)
-  (net 12 N-0000010)
-  (net 13 N-0000013)
-  (net 14 VCC)
+  (net 11 N-0000010)
+  (net 12 N-000002)
+  (net 13 N-000005)
+  (net 14 N-000006)
+  (net 15 N-000007)
+  (net 16 VCC)
   (net_class Default "This is the default net class."
     (clearance 0.2032)
@@
     (add_net /SENSE)
     (add_net /drain)
-    (add_net N-000001)
     (add_net N-0000010)
-    (add_net N-0000013)
+    (add_net N-000002)
+    (add_net N-000005)
+    (add_net N-000006)
+    (add_net N-000007)
   )
   (net_class Power ""
@@
     (pad 2 thru_hole oval (at -1.27 0.635 180) (size 1.05 1.5) (drill 0.5 (offset 0 0.2))
       (layers *.Cu *.Mask B.SilkS)
-      (net 14 VCC)
+      (net 16 VCC)
     )
     (pad 3 thru_hole oval (at 0 -0.635 180) (size 1.05 1.5) (drill 0.5 (offset 0 -0.2))
@@
     (pad 1 smd rect (at -0.94996 0) (size 1.29794 1.4986)
       (layers Front F.Mask)
-      (net 14 VCC)
+      (net 16 VCC)
     )
     (pad 2 smd rect (at 0.94996 0) (size 1.29794 1.4986)
@@
     (pad 1 smd rect (at -0.94996 0) (size 1.29794 1.4986)
       (layers Front F.Mask)
-      (net 14 VCC)
+      (net 16 VCC)
     )
     (pad 2 smd rect (at 0.94996 0) (size 1.29794 1.4986)
@@
     (pad 2 smd rect (at 0.84836 0 180) (size 0.99822 1.09982)
       (layers Front F.Mask)
-      (net 11 N-000001)
+      (net 13 N-000005)
     )
   )
@@
     (pad 1 smd rect (at -0.84836 0 180) (size 0.99822 1.09982)
       (layers Front F.Mask)
-      (net 13 N-0000013)
+      (net 12 N-000002)
     )
     (pad 2 smd rect (at 0.84836 0 180) (size 0.99822 1.09982)
       (layers Front F.Mask)
-      (net 12 N-0000010)
+      (net 11 N-0000010)
     )
   )
@@
     (pad 1 smd rect (at -0.94996 0 180) (size 1.29794 1.4986)
       (layers Front F.Mask)
-      (net 12 N-0000010)
+      (net 11 N-0000010)
     )
     (pad 2 smd rect (at 0.94996 0 180) (size 1.29794 1.4986)
@@
     (pad 1 smd rect (at -0.95 1.1 90) (size 1 1.4)
       (layers Front F.Mask)
-      (net 11 N-000001)
+      (net 13 N-000005)
     )
     (pad 2 smd rect (at 0.95 1.1 90) (size 1 1.4)
@@
     (pad 5 smd rect (at -0.95 -1.3) (size 0.65 1.25)
       (layers Front F.Mask)
-      (net 14 VCC)
+      (net 16 VCC)
     )
   )
@@
     (pad 3 smd rect (at 0.95 1.3 270) (size 0.65 1.25)
       (layers Front F.Mask)
-      (net 12 N-0000010)
+      (net 11 N-0000010)
     )
     (pad 4 smd rect (at 0.95 -1.3 270) (size 0.65 1.25)
@@
     (pad 5 smd rect (at -0.95 -1.3 270) (size 0.65 1.25)
       (layers Front F.Mask)
-      (net 14 VCC)
+      (net 16 VCC)
+    )
+  )
+  (module MADW__SOT23 (layer Front)
+    (at 99.175 65.15)
+    (descr "SMALL OUTLINE TRANSISTOR")
+    (tags "SMALL OUTLINE TRANSISTOR")
+    (attr smd)
+    (fp_text reference DS1 (at 0 -3) (layer F.SilkS)
+      (effects (font (size 1 1) (thickness 0.2)))
+    )
+    (fp_text value BAT54 (at 0 3.2) (layer F.SilkS)
+      (effects (font (size 1 1) (thickness 0.2)))
+    )
+    (fp_line (start 1.9 -2.2) (end 1.9 2.2) (layer F.SilkS) (width 0.2))
+    (fp_line (start 1.9 2.2) (end -1.9 2.2) (layer F.SilkS) (width 0.2))
+    (fp_line (start -1.9 2.2) (end -1.9 -2.2) (layer F.SilkS) (width 0.2))
+    (fp_line (start -1.9 -2.2) (end 1.9 -2.2) (layer F.SilkS) (width 0.2))
+    (fp_line (start -0.2286 -0.7112) (end 0.2286 -0.7112) (layer F.SilkS) (width 0.2))
+    (fp_line (start 0.2286 -0.7112) (end 0.2286 -1.29286) (layer F.SilkS) (width 0.2))
+    (fp_line (start -0.2286 -1.29286) (end 0.2286 -1.29286) (layer F.SilkS) (width 0.2))
+    (fp_line (start -0.2286 -0.7112) (end -0.2286 -1.29286) (layer F.SilkS) (width 0.2))
+    (fp_line (start 0.7112 1.29286) (end 1.1684 1.29286) (layer F.SilkS) (width 0.2))
+    (fp_line (start 1.1684 1.29286) (end 1.1684 0.7112) (layer F.SilkS) (width 0.2))
+    (fp_line (start 0.7112 0.7112) (end 1.1684 0.7112) (layer F.SilkS) (width 0.2))
+    (fp_line (start 0.7112 1.29286) (end 0.7112 0.7112) (layer F.SilkS) (width 0.2))
+    (fp_line (start -1.1684 1.29286) (end -0.7112 1.29286) (layer F.SilkS) (width 0.2))
+    (fp_line (start -0.7112 1.29286) (end -0.7112 0.7112) (layer F.SilkS) (width 0.2))
+    (fp_line (start -1.1684 0.7112) (end -0.7112 0.7112) (layer F.SilkS) (width 0.2))
+    (fp_line (start -1.1684 1.29286) (end -1.1684 0.7112) (layer F.SilkS) (width 0.2))
+    (fp_line (start -0.49784 0.29972) (end 0.49784 0.29972) (layer F.SilkS) (width 0.2))
+    (fp_line (start 0.49784 0.29972) (end 0.49784 -0.29972) (layer F.SilkS) (width 0.2))
+    (fp_line (start -0.49784 -0.29972) (end 0.49784 -0.29972) (layer F.SilkS) (width 0.2))
+    (fp_line (start -0.49784 0.29972) (end -0.49784 -0.29972) (layer F.SilkS) (width 0.2))
+    (fp_line (start 1.41986 -0.65786) (end 1.41986 0.65786) (layer F.SilkS) (width 0.2))
+    (fp_line (start 1.41986 0.65786) (end -1.41986 0.65786) (layer F.SilkS) (width 0.2))
+    (fp_line (start -1.41986 0.65786) (end -1.41986 -0.65786) (layer F.SilkS) (width 0.2))
+    (fp_line (start -1.41986 -0.65786) (end 1.41986 -0.65786) (layer F.SilkS) (width 0.2))
+    (pad 1 smd rect (at -0.95 1.1) (size 1 1.4)
+      (layers Front F.Mask)
+      (net 1 /CHARGE)
+    )
+    (pad 2 smd rect (at 0.95 1.1) (size 1 1.4)
+      (layers Front F.Mask)
+    )
+    (pad 3 smd rect (at 0 -1.1) (size 1 1.4)
+      (layers Front F.Mask)
+      (net 12 N-000002)
+    )
+  )
+  (module MADW__R0603_2 (layer Front)
+    (at 93.275 67.05)
+    (descr RESISTOR)
+    (tags RESISTOR)
+    (attr smd)
+    (fp_text reference R4 (at 0 -1.9) (layer F.SilkS)
+      (effects (font (size 1 1) (thickness 0.2)))
+    )
+    (fp_text value 500k (at 0 2.1) (layer F.SilkS)
+      (effects (font (size 1 1) (thickness 0.2)))
+    )
+    (fp_line (start -1.7 -0.9) (end 1.7 -0.9) (layer F.SilkS) (width 0.2))
+    (fp_line (start 1.7 -0.9) (end 1.7 0.9) (layer F.SilkS) (width 0.2))
+    (fp_line (start 1.7 0.9) (end -1.7 0.9) (layer F.SilkS) (width 0.2))
+    (fp_line (start -1.7 0.9) (end -1.7 -0.9) (layer F.SilkS) (width 0.2))
+    (fp_line (start 0.4318 0.4318) (end 0.8382 0.4318) (layer F.SilkS) (width 0.2))
+    (fp_line (start 0.8382 0.4318) (end 0.8382 -0.4318) (layer F.SilkS) (width 0.2))
+    (fp_line (start 0.4318 -0.4318) (end 0.8382 -0.4318) (layer F.SilkS) (width 0.2))
+    (fp_line (start 0.4318 0.4318) (end 0.4318 -0.4318) (layer F.SilkS) (width 0.2))
+    (fp_line (start -0.8382 0.4318) (end -0.4318 0.4318) (layer F.SilkS) (width 0.2))
+    (fp_line (start -0.4318 0.4318) (end -0.4318 -0.4318) (layer F.SilkS) (width 0.2))
+    (fp_line (start -0.8382 -0.4318) (end -0.4318 -0.4318) (layer F.SilkS) (width 0.2))
+    (fp_line (start -0.8382 0.4318) (end -0.8382 -0.4318) (layer F.SilkS) (width 0.2))
+    (fp_line (start -0.4318 0.3556) (end 0.4318 0.3556) (layer F.SilkS) (width 0.2))
+    (fp_line (start 0.4318 -0.3556) (end -0.4318 -0.3556) (layer F.SilkS) (width 0.2))
+    (pad 1 smd rect (at -0.84836 0) (size 0.99822 1.09982)
+      (layers Front F.Mask)
+      (net 11 N-0000010)
+    )
+    (pad 2 smd rect (at 0.84836 0) (size 0.99822 1.09982)
+      (layers Front F.Mask)
+      (net 9 GND)
     )
   )
@@
       (effects (font (size 1 1) (thickness 0.2)))
     )
-    (fp_text value ATTINY13A-MM (at 0 3.3) (layer F.SilkS)
-      (effects (font (size 1 1) (thickness 0.2)))
-    )
-    (fp_line (start 2.4 -1.9) (end -2.4 -1.9) (layer F.SilkS) (width 0.2))
-    (fp_line (start -2.4 -1.9) (end -2.4 1.9) (layer F.SilkS) (width 0.2))
+    (fp_text value MADW__ATTINY13-MM (at 0 3.3) (layer F.SilkS)
+      (effects (font (size 1 1) (thickness 0.2)))
+    )
+    (fp_line (start -2.4 -1.5) (end -2.4 1.9) (layer F.SilkS) (width 0.2))
+    (fp_line (start -2 -1.9) (end 2.4 -1.9) (layer F.SilkS) (width 0.2))
+    (fp_line (start -2 -1.9) (end -2.4 -1.5) (layer F.SilkS) (width 0.2))
     (fp_line (start 2.4 1.9) (end -2.4 1.9) (layer F.SilkS) (width 0.2))
     (fp_line (start 2.4 -1.9) (end 2.4 1.9) (layer F.SilkS) (width 0.2))
@@
     (pad 3 smd rect (at -1.5 0) (size 1 0.25)
       (layers Front F.Mask)
+      (net 14 N-000006)
     )
     (pad 4 smd rect (at -1.5 0.5) (size 1 0.25)
@@
     (pad 8 smd rect (at 1.5 0) (size 1 0.25)
       (layers Front F.Mask)
+      (net 15 N-000007)
     )
     (pad 9 smd rect (at 1.5 -0.5) (size 1 0.25)
@@
     (pad 10 smd rect (at 1.5 -1) (size 1 0.25)
       (layers Front F.Mask)
-      (net 14 VCC)
-    )
-    (pad 11 thru_hole rect (at 0 0) (size 1.75 2.7) (drill 0.5)
+      (net 16 VCC)
+    )
+    (pad PAD thru_hole rect (at 0 0) (size 1.75 2.7) (drill 0.5)
       (layers *.Cu *.Mask)
+      (net 9 GND)
     )
   )
@@
   (segment (start 99.74996 49.54996) (end 99.74996 49.6) (width 0.3048) (layer Front) (net 9) (status 30))
   (segment (start 99.7 49.5) (end 99.74996 49.54996) (width 0.3048) (layer Front) (net 9) (status 30))
-  (segment (start 97.7 51.84996) (end 97.85004 52) (width 0.3048) (layer Front) (net 14) (status 30))
+  (segment (start 97.7 51.84996) (end 97.85004 52) (width 0.3048) (layer Front) (net 16) (status 30))
 )

Commit message: Switch-timed: switched to ATtiny10 SOT23-6.
Parts:
- added R5: 1k, MADW__R0603_2, F.Cu at (89.4, 67.4)
- IC1: value MADW__ATTINY13-MM -> ATTINY10-TS; footprint MADW__MLF10 -> MADW__SOT23-6
- JP1: value ISP -> MADW__AVR_TPI
- R3: value 150R -> 1k
- moved DS1 6.17 mm to (105.2, 63.8)
- moved R4 3.27 mm to (95.5, 64.7)
- turned IC1 to 90 degrees
Connections:
- IC1 pad 1: /RESET -> /GATE
- IC1 pad 2: /SENSE -> GND
- IC1 pad 3: N-000006 -> /SENSE
- IC1 pad 5: GND -> VCC
- IC1 pad 6: /MOSI -> /RESET
- JP1 pad 1: /MISO -> /GATE
- JP1 pad 3: /SCK -> /SENSE
- JP1 pad 4: /MOSI -> N-000007
- R1 pad 2: /MOSI -> /GATE
- R2 pad 1: /MOSI -> /GATE
- U1 pad 1: /SENSE -> N-000002
- U1 pad 4: /SENSE -> N-000002

Commit message: Revert "Switch-timed: switched to ATtiny10 SOT23-6."
This reverts commit 7426c306dc58e77c9809db77e26f6b62b76c1d9c.

C + ATtiny10 not supported by avr-gcc
Parts:
- removed R5: 1k, MADW__R0603_2
- IC1: value ATTINY10-TS -> MADW__ATTINY13-MM; footprint MADW__SOT23-6 -> MADW__MLF10
- JP1: value MADW__AVR_TPI -> ISP
- R3: value 1k -> 150R
- moved DS1 6.17 mm to (99.2, 65.2)
- moved R4 3.27 mm to (93.3, 67.0)
- turned IC1 to 0 degrees
Connections:
- IC1 pad 1: /GATE -> /RESET
- IC1 pad 2: GND -> /SENSE
- IC1 pad 3: /SENSE -> N-000006
- IC1 pad 5: VCC -> GND
- IC1 pad 6: /RESET -> /MOSI
- JP1 pad 1: /GATE -> /MISO
- JP1 pad 3: /SENSE -> /SCK
- JP1 pad 4: N-000007 -> /MOSI
- R1 pad 2: /GATE -> /MOSI
- R2 pad 1: /GATE -> /MOSI
- U1 pad 1: N-000002 (its old number) -> /SENSE
- U1 pad 4: N-000002 (its old number) -> /SENSE
